Commit message: thresh of the detection set, working fine
In this version it do not have a more importance variable v1

File: transfer_carrier_description/urdf/transfer_carrier.urdf (robot description, URDF)
Before this commit: robot sam_bot, 3 links, 2 joints
Joints:
- joint hokuyo_joint: origin xyz=1.8 0.0 0.0 rpy=0 0 0 -> xyz=1.8 0.0 0.1 rpy=0 0 0

Commit message: lidar processing added add debbing of the wall

File: transfer_carrier_description/urdf/transfer_carrier.urdf (robot description, URDF)
Before this commit: robot sam_bot, 3 links, 2 joints
Links:
- added link detector_wall
Joints:
- added joint detector_wall_joint: type fixed, parent base_footprint, child detector_wall, origin xyz=2.0 0 0.3 rpy=0 0 0
